File: RX/Board/receiver.sch (KiCad schematic (older format))
At the start: 10 parts, among them J2 PROG_CONN, J3 RX_JMP, J4 TX_JMP, J5 AT_MODE_JUMP, J7 GENERIC, U1 ARDUINO_PRO_MINI, U2 ITEAD_HC-05

Commit message: Corrected bugs and added first prototype of receiver board
Parts:
- removed J5: AT_MODE_JUMP, Pin_Headers:Pin_Header_Straight_1x02, symbol CONN_01X02
- removed U2: ITEAD_HC-05, foots:HC-05, symbol ITEAD_HC-05
- added J5: LIGHTS, Pin_Headers:Pin_Header_Angled_1x06, symbol CONN_01X06
- added J6: Bluetooth, Pin_Headers:Pin_Header_Angled_1x04, symbol CONN_01X04
- added J8: BIG_BATTERY, Pin_Headers:Pin_Header_Angled_1x02, symbol CONN_01X02
- J1: renamed from J?; value CONN_01X03 -> ESC; footprint (none) -> Pin_Headers:Pin_Header_Angled_1x03
- J7: footprint Pin_Headers:Pin_Header_Straight_1x04 -> Pin_Headers:Pin_Header_Angled_1x04
Connections:
- net +BATT: now also J8.2 (P2); no longer J1.2 (P2), U1.27 (RAW)
- net G1: now also U1.19 (D13); no longer U1.12 (D9)
- net G2: now also U1.20 (A0); no longer U1.11 (D8)
- net G3: now also U1.21 (A1); no longer U1.10 (D7)
- net GNDREF: now also J5.1 (P1), J6.2 (P2), J8.1 (P1)
- net RX_BT: now also J6.4 (P4)
- net TX_BT: now also J6.3 (P3)
- net LIGHT_5: now reaches U1.8 (D5)
- net LIGHT_5: now also J5.6 (P6)
- net LIGHT_4: now reaches U1.9 (D6)
- net LIGHT_4: now also J5.5 (P5)
- net +3V3 renamed +5V
- net +5V: now also J1.2 (P2), J6.1 (P1)
- net AT_MODE: no longer names the net of U1.5 (D2)
- new net LIGHT_1: J5.2 (P2), U1.12 (D9)
- new net LIGHT_2: J5.3 (P3), U1.11 (D8)
- new net LIGHT_3: J5.4 (P4), U1.10 (D7)
- no-connect marks 40 -> 13
Other:
- note added: "Programming \nconnector\n"
- note added: "Programming jumper"
- note removed: "Connettore per\nprogrammazione\n"
- note removed: "Jumper per \nprogrammazione\n"
- note removed: "Jumper used for entering AT-MODE\n"
