File: TX/Board/controller.sch (KiCad schematic (older format))
At the start: 15 parts, among them J1 PRESENCE_SENS, J2 PROG_CONN, J3 RX_JMP, J4 TX_JMP, J5 AT_MODE_JUMP, J6 BATT_CONN, J7 GENERIC, U1 ARDUINO_PRO_MINI, U2 ITEAD_HC-05

Commit message: Added images and first version of the led panel
Parts:
- removed J7: GENERIC, Pin_Headers:Pin_Header_Straight_1x04, symbol CONN_01X04
- added J7: LED_SPEED, Pin_Headers:Pin_Header_Straight_1x11, symbol CONN_01X11
Connections:
- net GNDREF: now also J7.1 (P1); no longer R3.2
- net SPLED_0: now reaches U1.14 (A6)
- net SPLED_0: now also J7.2 (P2)
- net SPLED_1: now reaches U1.15 (A7)
- net SPLED_1: now also J7.3 (P3)
- net BATT_STAT: now reaches U1.19 (D13)
- net SPLED_9: now reaches U1.5 (D2)
- net SPLED_9: now also J7.11 (P11)
- net SPLED_8: now reaches U1.6 (D3)
- net SPLED_8: now also J7.10 (P10)
- net SPLED_7: now reaches U1.7 (D4)
- net SPLED_7: now also J7.9 (P9)
- net SPLED_6: now reaches U1.8 (D5)
- net SPLED_6: now also J7.8 (P8)
- net SPLED_5: now reaches U1.9 (D6)
- net SPLED_5: now also J7.7 (P7)
- net G1 renamed SPLED_2
- net SPLED_2: now also J7.4 (P4)
- net G2 renamed SPLED_3
- net SPLED_3: now also J7.5 (P5)
- net G3 renamed SPLED_4
- net SPLED_4: now also J7.6 (P6)
- no-connect marks 41 -> 33
Other:
- note removed: "Generic connector\n"
Changed lines of the file:
@@
 LIBS:arduino
 LIBS:00 LIBRARY
+LIBS:w_rtx
 LIBS:controller-cache
 EELAYER 25 0
@@
 $Descr A4 11693 8268
 encoding utf-8
-Sheet 1 1
+Sheet 1 2
 Title "handy - TX"
 Date "2017-03-29"
@@
 $EndDescr
 $Comp
-L ARDUINO_PRO_MINI U1
-U 1 1 58BE9155
-P 5850 3500
-F 0 "U1" H 5850 3050 50  0000 L CNN
-F 1 "ARDUINO_PRO_MINI" V 5750 3100 50  0000 L CNN
-F 2 "foots:Arduino_PRO_MINI" H 5950 3300 50  0001 C CNN
-F 3 "" H 5950 3300 50  0001 C CNN
-	1    5850 3500
-	1    0    0    -1
-$EndComp
-$Comp
 L ITEAD_HC-05 U2
 U 1 1 58BE9179
@@
 $EndComp
 $Comp
-L GNDREF #PWR6
+L GNDREF #PWR01
 U 1 1 58C7D630
 P 2100 4050
-F 0 "#PWR6" H 2100 3800 50  0001 C CNN
+F 0 "#PWR01" H 2100 3800 50  0001 C CNN
 F 1 "GNDREF" H 2100 3900 50  0000 C CNN
 F 2 "" H 2100 4050 50  0001 C CNN
@@
 $EndComp
 $Comp
-L +3.3V #PWR5
+L +3.3V #PWR02
 U 1 1 58C7D6CB
 P 2100 1500
-F 0 "#PWR5" H 2100 1350 50  0001 C CNN
+F 0 "#PWR02" H 2100 1350 50  0001 C CNN
 F 1 "+3.3V" H 2100 1640 50  0000 C CNN
 F 2 "" H 2100 1500 50  0001 C CNN
@@
 $EndComp
 $Comp
-L +3.3V #PWR11
+L +3.3V #PWR03
 U 1 1 58C7D6EC
 P 7050 1800
-F 0 "#PWR11" H 7050 1650 50  0001 C CNN
+F 0 "#PWR03" H 7050 1650 50  0001 C CNN
 F 1 "+3.3V" H 7050 1940 50  0000 C CNN
 F 2 "" H 7050 1800 50  0001 C CNN
@@
 $EndComp
 $Comp
-L GNDREF #PWR10
+L GNDREF #PWR04
 U 1 1 58C7D7DC
 P 6800 2950
-F 0 "#PWR10" H 6800 2700 50  0001 C CNN
+F 0 "#PWR04" H 6800 2700 50  0001 C CNN
 F 1 "GNDREF" H 6800 2800 50  0000 C CNN
 F 2 "" H 6800 2950 50  0001 C CNN
@@
 $EndComp
 $Comp
-L GNDREF #PWR7
+L GNDREF #PWR05
 U 1 1 58C7E1D0
 P 4200 7350
-F 0 "#PWR7" H 4200 7100 50  0001 C CNN
+F 0 "#PWR05" H 4200 7100 50  0001 C CNN
 F 1 "GNDREF" H 4200 7200 50  0000 C CNN
 F 2 "" H 4200 7350 50  0001 C CNN
@@
 $EndComp
 $Comp
-L +3.3V #PWR8
+L +3.3V #PWR06
 U 1 1 58C7E222
 P 4500 6400
-F 0 "#PWR8" H 4500 6250 50  0001 C CNN
+F 0 "#PWR06" H 4500 6250 50  0001 C CNN
 F 1 "+3.3V" H 4500 6540 50  0000 C CNN
 F 2 "" H 4500 6400 50  0001 C CNN
@@
 $EndComp
 $Comp
-L GNDREF #PWR2
+L GNDREF #PWR07
 U 1 1 58C7E432
 P 1150 5850
-F 0 "#PWR2" H 1150 5600 50  0001 C CNN
+F 0 "#PWR07" H 1150 5600 50  0001 C CNN
 F 1 "GNDREF" H 1150 5700 50  0000 C CNN
 F 2 "" H 1150 5850 50  0001 C CNN
@@
 $EndComp
 $Comp
-L +3.3V #PWR1
+L +3.3V #PWR08
 U 1 1 58C7E455
 P 1150 5000
-F 0 "#PWR1" H 1150 4850 50  0001 C CNN
+F 0 "#PWR08" H 1150 4850 50  0001 C CNN
 F 1 "+3.3V" H 1150 5140 50  0000 C CNN
 F 2 "" H 1150 5000 50  0001 C CNN
@@
 AT_MODE
 $Comp
-L +3.3V #PWR15
+L +3.3V #PWR09
 U 1 1 58D52A1F
 P 9750 1150
-F 0 "#PWR15" H 9750 1000 50  0001 C CNN
+F 0 "#PWR09" H 9750 1000 50  0001 C CNN
 F 1 "+3.3V" H 9750 1290 50  0000 C CNN
 F 2 "" H 9750 1150 50  0001 C CNN
@@
 $EndComp
 $Comp
-L +BATT #PWR9
+L +BATT #PWR010
 U 1 1 58D52B9C
 P 6450 2800
-F 0 "#PWR9" H 6450 2650 50  0001 C CNN
+F 0 "#PWR010" H 6450 2650 50  0001 C CNN
 F 1 "+BATT" H 6450 2940 50  0000 C CNN
 F 2 "" H 6450 2800 50  0001 C CNN
@@
 $EndComp
 $Comp
-L +BATT #PWR16
+L +BATT #PWR011
 U 1 1 58D52CB9
 P 10750 2100
-F 0 "#PWR16" H 10750 1950 50  0001 C CNN
+F 0 "#PWR011" H 10750 1950 50  0001 C CNN
 F 1 "+BATT" H 10750 2240 50  0000 C CNN
 F 2 "" H 10750 2100 50  0001 C CNN
@@
 $EndComp
 $Comp
-L GNDREF #PWR17
+L GNDREF #PWR012
 U 1 1 58D52DB0
 P 10750 2650
-F 0 "#PWR17" H 10750 2400 50  0001 C CNN
+F 0 "#PWR012" H 10750 2400 50  0001 C CNN
 F 1 "GNDREF" H 10750 2500 50  0000 C CNN
 F 2 "" H 10750 2650 50  0001 C CNN
@@
 $EndComp
 $Comp
-L +BATT #PWR13
+L +BATT #PWR013
 U 1 1 58D535FE
 P 9250 3450
-F 0 "#PWR13" H 9250 3300 50  0001 C CNN
+F 0 "#PWR013" H 9250 3300 50  0001 C CNN
 F 1 "+BATT" H 9250 3590 50  0000 C CNN
 F 2 "" H 9250 3450 50  0001 C CNN
@@
 	1    0    0    -1
 $EndComp
-$Comp
-L GNDREF #PWR14
-U 1 1 58D53630
-P 9250 4750
-F 0 "#PWR14" H 9250 4500 50  0001 C CNN
-F 1 "GNDREF" H 9250 4600 50  0000 C CNN
-F 2 "" H 9250 4750 50  0001 C CNN
-F 3 "" H 9250 4750 50  0001 C CNN
-	1    9250 4750
-	1    0    0    -1
-$EndComp
 Text GLabel 8900 4050 0    60   Input ~ 0
 BATT_SENS
@@
 Text Notes 8400 3650 0    60   ~ 0
 Battery charge\nreading\n
-NoConn ~ 5150 3750
-NoConn ~ 5150 3650
-NoConn ~ 5150 3550
 NoConn ~ 5500 2500
 NoConn ~ 6400 3850
@@
 NoConn ~ 1500 3000
 NoConn ~ 2700 2350
-NoConn ~ 5150 3250
-$Comp
-L CONN_01X04 J7
-U 1 1 58D58255
-P 8650 5800
-F 0 "J7" H 8650 6050 50  0000 C CNN
-F 1 "GENERIC" V 8750 5800 50  0000 C CNN
-F 2 "Pin_Headers:Pin_Header_Straight_1x04" H 8650 5800 50  0001 C CNN
-F 3 "" H 8650 5800 50  0001 C CNN
-	1    8650 5800
-	-1   0    0    1
-$EndComp
-$Comp
-L GNDREF #PWR12
-U 1 1 58D58378
-P 9050 6200
-F 0 "#PWR12" H 9050 5950 50  0001 C CNN
-F 1 "GNDREF" H 9050 6050 50  0000 C CNN
-F 2 "" H 9050 6200 50  0001 C CNN
-F 3 "" H 9050 6200 50  0001 C CNN
-	1    9050 6200
-	1    0    0    -1
-$EndComp
-Text GLabel 9150 5650 2    60   Input ~ 0
-G1
-Text GLabel 9150 5750 2    60   Input ~ 0
-G2
-Text GLabel 9150 5850 2    60   Input ~ 0
-G3
-Text GLabel 5150 4050 0    60   Input ~ 0
-G1
-Text GLabel 5150 3950 0    60   Input ~ 0
-G2
-Text GLabel 5150 3850 0    60   Input ~ 0
-G3
-Text Notes 8550 5500 0    60   ~ 0
-Generic connector\n
 Text GLabel 5700 2150 1    60   Input ~ 0
 RX_ARD
@@
 	2000 3600 2000 3850
 Wire Wire Line
-	9050 6200 9050 5950
-Wire Wire Line
-	9050 5950 8850 5950
-Wire Wire Line
-	9150 5650 8850 5650
-Wire Wire Line
-	8850 5750 9150 5750
-Wire Wire Line
-	8850 5850 9150 5850
-Wire Wire Line
 	6700 3450 6400 3450
-Wire Notes Line
-	8350 6400 9450 6400
-Wire Notes Line
-	9450 6400 9450 5300
-Wire Notes Line
-	9450 5300 8350 5300
-Wire Notes Line
-	8350 5300 8350 6400
 Text GLabel 5000 3050 0    60   Input ~ 0
 RX_ARD
@@
 Wire Wire Line
 	5000 2950 5150 2950
-Text GLabel 5000 3150 0    60   Input ~ 0
-RST_ARD
 Wire Wire Line
 	5150 3150 5000 3150
@@
 Text GLabel 6700 3550 2    60   Input ~ 0
 AT_MODE
-NoConn ~ 6400 3750
-NoConn ~ 5150 3450
 Wire Wire Line
 	6700 3550 6400 3550
@@
 $EndComp
 $Comp
-L +3.3V #PWR3
+L +3.3V #PWR014
 U 1 1 58E0B708
 P 1500 6700
-F 0 "#PWR3" H 1500 6550 50  0001 C CNN
+F 0 "#PWR014" H 1500 6550 50  0001 C CNN
 F 1 "+3.3V" H 1500 6840 50  0000 C CNN
 F 2 "" H 1500 6700 50  0001 C CNN
@@
 	1500 6800 1500 6700
 $Comp
-L GNDREF #PWR4
+L GNDREF #PWR015
 U 1 1 58E0B866
 P 1500 7450
-F 0 "#PWR4" H 1500 7200 50  0001 C CNN
+F 0 "#PWR015" H 1500 7200 50  0001 C CNN
 F 1 "GNDREF" H 1500 7300 50  0000 C CNN
 F 2 "" H 1500 7450 50  0001 C CNN
@@
 Wire Wire Line
 	6700 3650 6400 3650
-NoConn ~ 5150 3350
 Wire Wire Line
 	6650 2400 6650 3050
@@
 Wire Notes Line
 	2700 6300 2700 7650
-NoConn ~ 6050 4450
-NoConn ~ 5950 4450
+$Comp
+L CONN_01X11 J7
+U 1 1 58E4A4A4
+P 8550 5700
+F 0 "J7" H 8550 6300 50  0000 C CNN
+F 1 "LED_SPEED" V 8650 5700 50  0000 C CNN
+F 2 "Pin_Headers:Pin_Header_Straight_1x11" H 8550 5700 50  0001 C CNN
+F 3 "" H 8550 5700 50  0001 C CNN
+	1    8550 5700
+	-1   0    0    1
+$EndComp
+Text GLabel 5000 3150 0    60   Input ~ 0
+RST_ARD
 NoConn ~ 5850 4450
+$Comp
+L ARDUINO_PRO_MINI U1
+U 1 1 58BE9155
+P 5850 3500
+F 0 "U1" H 5850 3050 50  0000 L CNN
+F 1 "ARDUINO_PRO_MINI" V 5750 3100 50  0000 L CNN
+F 2 "foots:Arduino_PRO_MINI" H 5950 3300 50  0001 C CNN
+F 3 "" H 5950 3300 50  0001 C CNN
+	1    5850 3500
+	1    0    0    -1
+$EndComp
+NoConn ~ 5150 3250
+$Comp
+L GNDREF #PWR016
+U 1 1 58E4A7B4
+P 9000 6350
+F 0 "#PWR016" H 9000 6100 50  0001 C CNN
+F 1 "GNDREF" H 9000 6200 50  0000 C CNN
+F 2 "" H 9000 6350 50  0001 C CNN
+F 3 "" H 9000 6350 50  0001 C CNN
+	1    9000 6350
+	1    0    0    -1
+$EndComp
+Wire Wire Line
+	9000 6350 9000 6200
+Wire Wire Line
+	9000 6200 8750 6200
+Text GLabel 8750 6100 2    60   Input ~ 0
+SPLED_0
+Text GLabel 8750 6000 2    60   Input ~ 0
+SPLED_1
+Text GLabel 8750 5900 2    60   Input ~ 0
+SPLED_2
+Text GLabel 8750 5800 2    60   Input ~ 0
+SPLED_3
+Text GLabel 8750 5700 2    60   Input ~ 0
+SPLED_4
+Text GLabel 8750 5600 2    60   Input ~ 0
+SPLED_5
+Text GLabel 8750 5500 2    60   Input ~ 0
+SPLED_6
+Text GLabel 8750 5400 2    60   Input ~ 0
+SPLED_7
+Text GLabel 8750 5300 2    60   Input ~ 0
+SPLED_8
+Text GLabel 8750 5200 2    60   Input ~ 0
+SPLED_9
+Text GLabel 5950 4450 3    60   Input ~ 0
+SPLED_0
+Text GLabel 6050 4450 3    60   Input ~ 0
+SPLED_1
+Text GLabel 5150 4050 0    60   Input ~ 0
+SPLED_2
+Text GLabel 5150 3950 0    60   Input ~ 0
+SPLED_3
+Text GLabel 5150 3850 0    60   Input ~ 0
+SPLED_4
+Text GLabel 5150 3750 0    60   Input ~ 0
+SPLED_5
+Text GLabel 5150 3650 0    60   Input ~ 0
+SPLED_6
+Text GLabel 5150 3550 0    60   Input ~ 0
+SPLED_7
+Text GLabel 5150 3450 0    60   Input ~ 0
+SPLED_8
+Text GLabel 5150 3350 0    60   Input ~ 0
+SPLED_9
+$Sheet
+S 8950 2300 800  600
+U 58E63085
+F0 "battery_charger" 60
+F1 "battery_charger.sch" 60
+$EndSheet
+Text GLabel 6700 3750 2    60   Input ~ 0
+BATT_STAT
+Wire Wire Line
+	6700 3750 6400 3750
 $EndSCHEMATC
